File: hardware/bassberry/pi.kicad_sch (KiCad schematic)
At the start: 13 parts, among them J101 RPi 40-pin (face-down socket), U101 24C32 (HAT ID)

Commit message: rev 0.2 board: routed with srouter, DRC 0 errors / 0 unconnected / 0 parity, digital twin 1-4 PASS; KiCad files, reports, renders
Parts:
- added C104: 100n, Capacitor_SMD:C_0603_1608Metric, symbol Device:C
- added Q101: DMP3013SFV, Package_SON:Diodes_PowerDI3333-8, symbol Transistor_FET:DMP3013SFV
- added Q102: DMMT5401, Package_TO_SOT_SMD:SOT-23-6, symbol Transistor_BJT:DMMT5401
- added R108: 10k 1%, Resistor_SMD:R_0603_1608Metric, symbol Device:R
- added R109: 47k 1%, Resistor_SMD:R_0603_1608Metric, symbol Device:R
- added TP101: ID_WP, TestPoint:TestPoint_Pad_D1.5mm, symbol Connector:TestPoint
- R107: value 10k -> 1k
- U101: value 24C32 (HAT ID) -> CAT24C32WI-GT3
Connections:
- net +3V3: now also C104.1
- net +5V: now also Q101.1 (S), Q101.2 (S), Q101.3 (S), Q102.5 (E2)
- net GND: now also C104.2, R108.2, R109.2
- net ID_WP: now also TP101.1
- net AMP2_PDN: now reaches J101.29 (GPCLK1/GPIO05)
- new net +5V_BUCK: Q101.5 (D), Q102.6 (E1)
- new net ZVD_B: Q102.1 (C1), Q102.2 (B1), Q102.3 (B2), R108.1
- new net ZVD_G: Q101.4 (G), Q102.4 (C2), R109.1
- no-connect marks 15 -> 14
Other:
- note added: "Back-power ideal diode (HAT design guide): +5V_BUCK -> +5V (Pi). 5 A rated: DMP3013SFV instead of DMG2305UX."
- note added: "HAT+ ID EEPROM @0x50 (CAT24C32). Write: bridge JP1, then eepflash.sh -w -t=24c32 -a=50 -f=bassberry.eep"
