File: hardware/bassberry/power.kicad_sch (KiCad schematic)
At the start: 79 parts, among them J301 USB-C (charge + console), Q301 40V N-MOS 5mR (AER4061BE equi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, Q302 40V N-MOS 5mR (AER4061BE equi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, Q303 40V N-MOS 5mR (AER4061BE equi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, Q304 40V N-MOS 5mR (AER4061BE equi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, Q305 30V N-MOS (RU3030M2) opt., SW301 PWRBANK (optional), U301 USBLC6-2SC6, U302 IP2366, U303 TPS565208, U304 MT3608, U305 HT7533-1, U306 HT7533-1

Commit message: rev 0.2 board: routed with srouter, DRC 0 errors / 0 unconnected / 0 parity, digital twin 1-4 PASS; KiCad files, reports, renders
Parts:
- removed JP301: PVDD_SUB select, Jumper:SolderJumper-3_P1.3mm_Bridged12_RoundedPad1.0x1.5mm, symbol Jumper:SolderJumper_3_Bridged12
- added R344: 0R 2512 (PVDD_SUB = battery), Resistor_SMD:R_2512_6332Metric, symbol Device:R
- added R345: DNP 0R 2512 (PVDD_SUB = boost), Resistor_SMD:R_2512_6332Metric, symbol Device:R
- U302: footprint Package_DFN_QFN:QFN-40-1EP_5x5mm_P0.4mm_EP3.6x3.6mm -> Package_DFN_QFN:QFN-40-1EP_5x5mm_P0.4mm_EP3.6x3.6mm_ThermalVias
- U306: value HT7533-1 -> XC6216B332PR; footprint Package_TO_SOT_SMD:SOT-89-3 -> Package_TO_SOT_SMD:SOT-89-5; symbol Regulator_Linear:HT75xx-1-SOT89 -> bassberry:XC6216B332PR
Connections:
- net +3V3_USB: now also U306.1 (VOUT); no longer U306.3 (VOUT)
- net +BATT: now also R344.1
- net BOOST_OUT: now also R345.1
- net GND: now also U306.2 (VSS); no longer U306.1 (GND)
- net PVDD_SUB: now also R344.2, R345.2
- net VBUS: now also U306.3 (CE), U306.5 (VIN); no longer U306.2 (VIN)
- net +5V renamed +5V_BUCK
Other:
- note added: "Pi 5V buck (+5V_BUCK, feeds the Pi through the back-power ideal diode on the Pi sheet): Vout = 0.76*(1+R31/R32) = 5.14 V. EN driven by supervisor (PI_PWR_EN)."
- note added: "Sub PVDD boost (optional): Vout = 0.6*(1+R41/R42) = 17.1 V. R44 (fitted) feeds PVDD_SUB from +BATT, R45 instead from the boost."
- note removed: "Pi 5V buck: Vout = 0.76*(1+R31/R32) = 5.14 V. EN driven by supervisor (PI_PWR_EN)."
- note removed: "Sub PVDD boost (optional): Vout = 0.6*(1+R41/R42) = 17.1 V. JP1 selects PVDD_SUB = +BATT (default) or boost."
